File: RGB LED Driver.kicad_sch (KiCad schematic)
At the start: 0 parts

Commit message: laid out stuff
Parts:
- added TP5 (x4): 5269 (Purple), TestPoint:TestPoint_Keystone_5000-5004_Miniature, symbol Connector:TestPoint_Alt
Connections:
- net ESP32/LED_B: now also TP5.1
- net ESP32/LED_G: now also TP5.1
- net ESP32/LED_R: now also TP5.1
- net ESP32/LED_W: now also TP5.1
Changed lines of the file:
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@@
 (kicad_sch (version 20230121) (generator eeschema)
-  (paper "A4")
+  (paper "USLetter")
+  (title_block
+    (date "2024-01-01")
+    (rev "A01")
+  )
+  (junction (at 196.85 102.87) (diameter 0) (color 0 0 0 0)
+  )
+  (junction (at 185.42 59.69) (diameter 0) (color 0 0 0 0)
+  )
+  (junction (at 194.31 137.16) (diameter 0) (color 0 0 0 0)
+  )
+  (junction (at 184.15 36.83) (diameter 0) (color 0 0 0 0)
+  )
   (wire (pts (xy 151.765 132.08) (xy 151.765 104.14))
     (stroke (width 0) (type default))
@@
     (stroke (width 0) (type default))
   )
-  (wire (pts (xy 194.945 102.87) (xy 200.025 102.87))
-    (stroke (width 0) (type default))
-  )
-  (wire (pts (xy 189.23 137.16) (xy 200.025 137.16))
+  (wire (pts (xy 194.31 137.16) (xy 200.025 137.16))
+    (stroke (width 0) (type default))
+  )
+  (wire (pts (xy 194.945 102.87) (xy 196.85 102.87))
+    (stroke (width 0) (type default))
+  )
+  (wire (pts (xy 189.23 137.16) (xy 194.31 137.16))
     (stroke (width 0) (type default))
   )
@@
     (stroke (width 0) (type default))
   )
+  (wire (pts (xy 196.85 102.87) (xy 200.025 102.87))
+    (stroke (width 0) (type default))
+  )
   (wire (pts (xy 234.95 138.43) (xy 245.11 138.43))
     (stroke (width 0) (type default))
@@
     (stroke (width 0) (type default))
   )
-  (wire (pts (xy 153.035 59.69) (xy 200.025 59.69))
+  (wire (pts (xy 184.15 36.83) (xy 200.025 36.83))
+    (stroke (width 0) (type default))
+  )
+  (wire (pts (xy 153.035 59.69) (xy 185.42 59.69))
     (stroke (width 0) (type default))
   )
@@
     (stroke (width 0) (type default))
   )
+  (wire (pts (xy 185.42 59.69) (xy 200.025 59.69))
+    (stroke (width 0) (type default))
+  )
   (wire (pts (xy 39.37 133.35) (xy 39.37 103.505))
     (stroke (width 0) (type default))
@@
     (stroke (width 0) (type default))
   )
-  (wire (pts (xy 148.59 36.83) (xy 200.025 36.83))
+  (wire (pts (xy 148.59 36.83) (xy 184.15 36.83))
     (stroke (width 0) (type default))
   )
@@
   (wire (pts (xy 114.935 48.26) (xy 119.38 48.26))
     (stroke (width 0) (type default))
+  )
+  (symbol (lib_id "Connector:TestPoint_Alt") (at 185.42 59.69 0) (unit 1)
+    (in_bom yes) (on_board yes) (dnp no) (fields_autoplaced)
+    (property "Reference" "TP5" (at 187.96 55.118 0)
+      (effects (font (size 1.27 1.27)) (justify left))
+    )
+    (property "Value" "5269 (Purple)" (at 187.96 57.658 0)
+      (effects (font (size 1.27 1.27)) (justify left))
+    )
+    (property "Footprint" "TestPoint:TestPoint_Keystone_5000-5004_Miniature" (at 190.5 59.69 0)
+      (effects (font (size 1.27 1.27)) hide)
+    )
+    (property "Datasheet" "~" (at 190.5 59.69 0)
+      (effects (font (size 1.27 1.27)) hide)
+    )
+    (property "Digikey PN" "" (at 185.42 59.69 0)
+      (effects (font (size 1.27 1.27)) hide)
+    )
+    (pin "1")
+    (instances
+      (project "RGB LED Driver"
+        (path "/955dc1f6-0512-416a-b86b-95ec08ff77cb/ecc56fd3-dc72-490a-a501-0be3de98d0c1"
+          (reference "TP5") (unit 1)
+        )
+        (path "/955dc1f6-0512-416a-b86b-95ec08ff77cb"
+          (reference "TP6") (unit 1)
+        )
+      )
+    )
+  )
+  (symbol (lib_id "Connector:TestPoint_Alt") (at 194.31 137.16 0) (unit 1)
+    (in_bom yes) (on_board yes) (dnp no) (fields_autoplaced)
+    (property "Reference" "TP5" (at 196.85 132.588 0)
+      (effects (font (size 1.27 1.27)) (justify left))
+    )
+    (property "Value" "5269 (Purple)" (at 196.85 135.128 0)
+      (effects (font (size 1.27 1.27)) (justify left))
+    )
+    (property "Footprint" "TestPoint:TestPoint_Keystone_5000-5004_Miniature" (at 199.39 137.16 0)
+      (effects (font (size 1.27 1.27)) hide)
+    )
+    (property "Datasheet" "~" (at 199.39 137.16 0)
+      (effects (font (size 1.27 1.27)) hide)
+    )
+    (property "Digikey PN" "" (at 194.31 137.16 0)
+      (effects (font (size 1.27 1.27)) hide)
+    )
+    (pin "1")
+    (instances
+      (project "RGB LED Driver"
+        (path "/955dc1f6-0512-416a-b86b-95ec08ff77cb/ecc56fd3-dc72-490a-a501-0be3de98d0c1"
+          (reference "TP5") (unit 1)
+        )
+        (path "/955dc1f6-0512-416a-b86b-95ec08ff77cb"
+          (reference "TP8") (unit 1)
+        )
+      )
+    )
   )
   (symbol (lib_id "power:+36V") (at 119.38 48.26 0) (unit 1)
@@
         )
       )
+    )
+  )
+  (symbol (lib_id "Connector:TestPoint_Alt") (at 196.85 102.87 0) (unit 1)
+    (in_bom yes) (on_board yes) (dnp no) (fields_autoplaced)
+    (property "Reference" "TP5" (at 199.39 98.298 0)
+      (effects (font (size 1.27 1.27)) (justify left))
+    )
+    (property "Value" "5269 (Purple)" (at 199.39 100.838 0)
+      (effects (font (size 1.27 1.27)) (justify left))
+    )
+    (property "Footprint" "TestPoint:TestPoint_Keystone_5000-5004_Miniature" (at 201.93 102.87 0)
+      (effects (font (size 1.27 1.27)) hide)
+    )
+    (property "Datasheet" "~" (at 201.93 102.87 0)
+      (effects (font (size 1.27 1.27)) hide)
+    )
+    (property "Digikey PN" "" (at 196.85 102.87 0)
+      (effects (font (size 1.27 1.27)) hide)
+    )
+    (pin "1")
+    (instances
+      (project "RGB LED Driver"
+        (path "/955dc1f6-0512-416a-b86b-95ec08ff77cb/ecc56fd3-dc72-490a-a501-0be3de98d0c1"
+          (reference "TP5") (unit 1)
+        )
+        (path "/955dc1f6-0512-416a-b86b-95ec08ff77cb"
+          (reference "TP7") (unit 1)
+        )
+      )
+    )
+  )
+  (symbol (lib_id "Connector:TestPoint_Alt") (at 184.15 36.83 0) (unit 1)
+    (in_bom yes) (on_board yes) (dnp no) (fields_autoplaced)
+    (property "Reference" "TP5" (at 186.69 32.258 0)
+      (effects (font (size 1.27 1.27)) (justify left))
+    )
+    (property "Value" "5269 (Purple)" (at 186.69 34.798 0)
+      (effects (font (size 1.27 1.27)) (justify left))
+    )
+    (property "Footprint" "TestPoint:TestPoint_Keystone_5000-5004_Miniature" (at 189.23 36.83 0)
+      (effects (font (size 1.27 1.27)) hide)
+    )
+    (property "Datasheet" "~" (at 189.23 36.83 0)
+      (effects (font (size 1.27 1.27)) hide)
+    )
+    (property "Digikey PN" "" (at 184.15 36.83 0)
+      (effects (font (size 1.27 1.27)) hide)
+    )
+    (pin "1")
+    (instances
+      (project "RGB LED Driver"
+        (path "/955dc1f6-0512-416a-b86b-95ec08ff77cb/ecc56fd3-dc72-490a-a501-0be3de98d0c1"
+          (reference "TP5") (unit 1)
+        )
+        (path "/955dc1f6-0512-416a-b86b-95ec08ff77cb"
+          (reference "TP5") (unit 1)
+        )
+      )

Commit message: neat-ified schematics
Connections:
- net ESP32/LED_B renamed BSig
- net ESP32/LED_G renamed GSig
- net ESP32/LED_R renamed RSig
- net ESP32/LED_W renamed WSig
Other:
- company: (none) -> The Art and Science of PCB Design
- title: (none) -> RGB LED Driver Demo Board
- moved on the sheet: TP5

Commit message: added digikey PNs
Parts:
- TP5: Digikey PN (none) -> 36-5269-ND; MPN (none) -> 5269
Changed lines of the file:
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@@
       (effects (font (size 1.27 1.27)) hide)
     )
-    (property "Digikey PN" "" (at 159.385 66.04 0)
+    (property "Digikey PN" "36-5269-ND" (at 159.385 66.04 0)
+      (effects (font (size 1.27 1.27)) hide)
+    )
+    (property "MPN" "5269" (at 159.385 66.04 0)
       (effects (font (size 1.27 1.27)) hide)
     )
@@
       (effects (font (size 1.27 1.27)) hide)
     )
-    (property "Digikey PN" "" (at 160.02 143.51 0)
+    (property "Digikey PN" "36-5269-ND" (at 160.02 143.51 0)
+      (effects (font (size 1.27 1.27)) hide)
+    )
+    (property "MPN" "5269" (at 160.02 143.51 0)
       (effects (font (size 1.27 1.27)) hide)
     )
@@
       (effects (font (size 1.27 1.27)) hide)
     )
-    (property "Digikey PN" "" (at 160.02 109.22 0)
+    (property "Digikey PN" "36-5269-ND" (at 160.02 109.22 0)
+      (effects (font (size 1.27 1.27)) hide)
+    )
+    (property "MPN" "5269" (at 160.02 109.22 0)
       (effects (font (size 1.27 1.27)) hide)
     )
@@
       (effects (font (size 1.27 1.27)) hide)
     )
-    (property "Digikey PN" "" (at 159.385 43.18 0)
+    (property "Digikey PN" "36-5269-ND" (at 159.385 43.18 0)
       (effects (font (size 1.27 1.27)) hide)
     )
+    (property "MPN" "5269" (at 159.385 43.18 0)
+      (effects (font (size 1.27 1.27)) hide)
+    )
