File: led_string.kicad_sch (KiCad schematic)
At the start: 11 parts

Commit message: neat-ified schematics
Other:
- company: (none) -> The Art and Science of PCB Design
- title: (none) -> RGB LED Driver Demo Board
Changed lines of the file:
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@@
   (paper "USLetter")
   (title_block
+    (title "RGB LED Driver Demo Board")
     (date "2024-01-01")
     (rev "A01")
+    (company "The Art and Science of PCB Design")
   )
   (wire (pts (xy 120.65 74.295) (xy 117.475 74.295))

Commit message: added digikey PNs
Parts:
- R24: MPN (none) -> 0805W8F0000
Changed lines of the file:
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@@
+      (effects (font (size 1.27 1.27)) hide)
+    )
+    (property "MPN" "0805W8F0000" (at 37.465 74.295 0)
       (effects (font (size 1.27 1.27)) hide)
     )

Commit message: added digikey PNs to all devices
Parts:
- R24: Digikey PN (none) -> RMCF0805ZT0R00CT-ND; MPN 0805W8F0000 -> RMCF0805FT0R00
Changed lines of the file:
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@@
       (effects (font (size 1.27 1.27)) hide)
     )
-    (property "Digikey PN" "" (at 37.465 74.295 0)
+    (property "Digikey PN" "RMCF0805ZT0R00CT-ND" (at 37.465 74.295 0)
       (effects (font (size 1.27 1.27)) hide)
     )
-    (property "MPN" "0805W8F0000" (at 37.465 74.295 0)
+    (property "MPN" "RMCF0805FT0R00" (at 37.465 74.295 0)
       (effects (font (size 1.27 1.27)) hide)
     )
