File: esp32.kicad_sch (KiCad schematic)
At the start: 14 parts, among them J2 Conn_01x06_Pin, J3 Conn_01x03_Pin, SW1 BOOT, U6 ESP32-WROOM-32, U7 CMXT3904

Commit message: cost reduction in BOM
Parts:
- C11, C16: Digikey PN 1276-1003-1-ND -> 1276-1029-1-ND; MPN CL21B104KBCNNNC -> CL21B105KBFNNNE
Changed lines of the file:
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@@
       (effects (font (size 1.27 1.27)) hide)
     )
-    (property "Digikey PN" "1276-1003-1-ND" (at 96.52 48.26 0)
-      (effects (font (size 1.27 1.27)) hide)
-    )
-    (property "MPN" "CL21B104KBCNNNC" (at 96.52 48.26 0)
+    (property "Digikey PN" "1276-1029-1-ND" (at 96.52 48.26 0)
+      (effects (font (size 1.27 1.27)) hide)
+    )
+    (property "MPN" "CL21B105KBFNNNE" (at 96.52 48.26 0)
       (effects (font (size 1.27 1.27)) hide)
     )
@@
       (effects (font (size 1.27 1.27)) hide)
     )
-    (property "Digikey PN" "1276-1003-1-ND" (at 39.37 60.96 0)
-      (effects (font (size 1.27 1.27)) hide)
-    )
-    (property "MPN" "CL21B104KBCNNNC" (at 39.37 60.96 0)
-      (effects (font (size 1.27 1.27)) hide)
-    )
+    (property "Digikey PN" "1276-1029-1-ND" (at 39.37 60.96 0)
+      (effects (font (size 1.27 1.27)) hide)
+    )
+    (property "MPN" "CL21B105KBFNNNE" (at 39.37 60.96 0)
+      (effects (font (size 1.27 1.27)) hide)
+    )

Commit message: [A02] Edited resistor values
R11 to 51K to allow for auto reset
R3 to 270K for 34V output
Parts:
- R11: value 10K -> 51K; Digikey PN RMCF0805FT10K0CT-ND -> RMCF0805FT51K0CT-ND
Other:
- note added: "A01: R11 = 10K A02: R11 = 51K"
Changed lines of the file:
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@@
     (stroke (width 0) (type default))
+  )
+  (text "A01: R11 = 10K\nA02: R11 = 51K" (at 31.75 41.91 0)
+    (effects (font (size 1.27 1.27)) (justify left bottom))
   )
   (text "BOM only - jumper for FTDI VIN select" (at 191.77 26.67 0)
@@
       (effects (font (size 1.27 1.27)) (justify left))
     )
-    (property "Value" "10K" (at 41.91 54.61 0)
+    (property "Value" "51K" (at 41.91 54.61 0)
       (effects (font (size 1.27 1.27)) (justify left))
     )
@@
       (effects (font (size 1.27 1.27)) hide)
     )
-    (property "Digikey PN" "RMCF0805FT10K0CT-ND" (at 39.37 53.34 0)
+    (property "Digikey PN" "RMCF0805FT51K0CT-ND" (at 39.37 53.34 0)
       (effects (font (size 1.27 1.27)) hide)
     )
